File: Rabid.kicad_pcb (KiCad board)
At the start: 2 copper layers, 344.6 x 122 mm, 192 parts, among them J1 USB Header, SW1 Esc, SW10 A, SW102 →, SW11 Z, SW12 LMeta, SW13 F1, SW14 2, SW15 W, SW16 S, SW17 X, SW18 LAlt, SW19 F2, SW2 Tilde, SW20 3, SW21 E, SW22 D, SW23 C, SW25 F3, SW26 4, SW27 R, SW28 F, SW29 V, SW3 Tab, SW31 F4, SW32 5, SW33 T, SW34 G, SW35 B, SW37 F5, SW38 6, SW39 Y, SW4 CapsLk, SW40 H, SW41 N, SW42 Space, SW43 F6, SW44 7, SW45 U, SW46 J, SW47 M, SW49 F7, SW5 LShift, SW50 8, SW51 I, SW52 K, SW53 ,, SW55 F8, SW56 9, SW57 O, SW58 L, SW59 ., SW6 LCtrl, SW61 F9, SW62 0, SW63 P, SW64 ;, SW65 /, SW66 AltGr, SW67 F10, SW68 -, SW69 [, SW70 ", SW71 RShift, SW72 RMeta, SW73 F11, SW74 =, SW75 ], SW76 ↲, SW78 Fn, SW79 F12, SW8 1, SW80 BkSpc, SW81 \, SW84 RCtrl, SW85 PrtSc, SW86 Ins, SW87 Del, SW9 Q, SW90 ←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

Commit message: Route columns. Board is now fully routed.
Routing:
- net ColA: track 126.0 -> 413.2 mm
- net ColB: track 100.3 -> 364.4 mm
- net ColC: track 121.2 -> 366.4 mm
- net ColD: track 99.3 -> 326.4 mm
- net ColE: track 96.1 -> 305.1 mm
- net ColF: track 96.1 -> 273.4 mm
- net ColG: track 127.6 -> 286.6 mm
- net ColH: track 99.1 -> 241.3 mm
- net ColI: track 99.6 -> 222.4 mm
- net ColN: track 73.4 -> 170.7 mm, vias 0 -> 1
- net ColJ: track 99.3 -> 188.5 mm
- net ColK: track 134.7 -> 205.8 mm
- net ColO: track 50.5 -> 115.7 mm, vias 0 -> 1
- net ColL: track 138.5 -> 194.0 mm
- net ColM: track 123.2 -> 173.3 mm, vias 0 -> 1
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