File: Rabid.kicad_pcb (KiCad board)
At the start: 2 copper layers, 343.4 x 121.9 mm, 193 parts, among them J1 USB Connector, J3 GPIO Debug Header, SW1 Esc, SW10 A, SW102 →, SW103 BootSel Switch, SW104 Reset Switch, SW11 Z, SW12 LMeta, SW13 F1, SW14 2, SW15 W, SW16 S, SW17 X, SW18 LAlt, SW19 F2, SW2 Tilde, SW20 3, SW21 E, SW22 D, SW23 C, SW25 F3, SW26 4, SW27 R, SW28 F, SW29 V, SW3 Tab, SW31 F4, SW32 5, SW33 T, SW34 G, SW35 B, SW37 F5, SW38 6, SW39 Y, SW4 CapsLk, SW40 H, SW41 N, SW42 Space, SW43 F6, SW44 7, SW45 U, SW46 J, SW47 M, SW49 F7, SW5 LShift, SW50 8, SW51 I, SW52 K, SW53 ,, SW55 F8, SW56 9, SW57 O, SW58 L, SW59 ., SW6 LCtrl, SW61 F9, SW62 0, SW63 P, SW64 ;, SW65 /, SW66 AltGr, SW67 F10, SW68 -, SW69 [, SW70 ", SW71 RShift, SW72 RMeta, SW73 F11, SW74 =, SW75 ], SW76 ↲, SW78 Fn, SW79 F12, SW8 1, SW80 BkSpc, SW81 \, SW84 RCtrl, SW85 PrtSc, SW86 Ins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

Commit message: Make Filco mounting hole smaller.
 - Add logo under spacebar.
 - Change PCB colour to black.
Parts:
- added G1: LOGO, RabidKeyboard:RabidKeyboardLogo, F.Cu at (141.0, 186.9)
- H3: value MountingHole_8.2mm -> MountingHole_4mm; footprint RabidKeyboard:MountingHole_8.2mm -> RabidKeyboard:MountingHole_4mm
- moved H3 0.76 mm to (212.1, 99.8)
Other:
- board text added: "BootSel"
- board text added: "Reset"

Commit message: Change RP2040 Stamp footprint to throughhole.
This ismore versatile as it allows either SMD or soldering on 2mm
pinheaders to use as a socket.
Parts:
- U1: footprint RP2040_Stamp:RP2040_Stamp_SMD -> RP2040_Stamp:RP2040_Stamp_THT
- moved G1 0.57 mm to (141.2, 186.4)
Routing:
- net GND: track 500.5 -> 531.8 mm, vias 2 -> 1
- net +5V: track 115.7 -> 120.5 mm, vias 1 -> 0
- net ColO: track 115.0 -> 119.3 mm, vias 1 -> 0
- net Row1: track 299.5 -> 303.4 mm, vias 1 -> 0
- net ColK: track 205.8 -> 209.6 mm
- net Row0: track 360.0 -> 357.2 mm, vias 1 -> 0
- net /USB_D-: track 67.9 -> 69.0 mm, vias 1 -> 0
- net /USB_D+: track 66.9 -> 67.9 mm, vias 1 -> 0
- net /~{RESET}: track 109.3 -> 110.2 mm, vias 2 -> 1
- net Row2: track 295.2 -> 294.5 mm, vias 1 -> 0
- net /BOOTSEL: track 93.1 -> 93.6 mm, vias 2 -> 1

Commit message: Make the power traces .7mm because I'm paranoid.
Parts:
- moved R2 2.03 mm to (354.3, 149.4)
- moved R1 2.03 mm to (354.3, 152.9)
- moved R3 2.03 mm to (354.3, 145.8)
Routing:
- net /CapsLED: track 405.9 -> 410.0 mm
- net +5V: track 120.5 -> 117.8 mm
- net /FnLED: track 181.4 -> 183.4 mm
- net /ScrollLED: track 70.5 -> 72.4 mm
- net GND: track 531.8 -> 530.3 mm
- net Row0: track 357.2 -> 358.2 mm
- net /USB_D-: track 69.0 -> 68.1 mm
- net /USB_D+: track 67.9 -> 67.1 mm
- net /CapsLED_GPIO: track 13.9 -> 14.4 mm

Commit message: Swap GPIO20 and GPIO21 (ROW0) pins.
The RP2040 Stamp has a WS2812B LED on the GPIO21 line.
It does have a jumper to disable the LED, but better to just work
around it, so it remains usable.
Connections:
- J3 pad 6: /GPIO20 -> /GPIO21
- U1 pad 21: /GPIO20 -> Row0
- U1 pad 22: Row0 -> /GPIO21
Routing:
- net /GPIO21: track 0.00 -> 38.8 mm
- net /GPIO20: track 36.3 -> 0.00 mm
- net ColN: track 169.5 -> 157.9 mm
- net Row0: track 358.2 -> 352.0 mm
- net /BOOTSEL: track 93.6 -> 98.5 mm
- net /~{RESET}: track 110.2 -> 114.8 mm
- net ColL: track 203.0 -> 199.1 mm
- net GND: track 530.3 -> 531.9 mm
- net +5V: track 117.8 -> 119.3 mm
Other:
- board text added: "GP21"
- board text removed: "GP20"

Commit message: Change Filco hole from 4mm to 5mm.
 - Rename FnLock to MetaLock.
 - Minor silkscreen changes.
Parts:
- D104: value CapsTopLED -> CapsLock
- D106: value ScrollTopLED -> ScrollLock
- D108: value FnTopLED -> MetaLock
- H3: value MountingHole_4mm -> MountingHole_5mm; footprint RabidKeyboard:MountingHole_4mm -> RabidKeyboard:MountingHole_5mm
- SW103: value BootSel Switch -> BootSel
- SW104: value Reset Switch -> Reset
Connections:
- net /FnLED renamed /MetaLED
- net /FnLED_GPIO renamed /MetaLED_GPIO
