File: pcb/Rabid.kicad_pcb (KiCad board)
At the start: 2 copper layers, 343.4 x 121.9 mm, 194 parts, among them J1 USB Connector, J3 GPIO Debug Header, SW1 Esc, SW10 A, SW102 →, SW103 BootSel, SW104 Reset, SW11 Z, SW12 LMeta, SW13 F1, SW14 2, SW15 W, SW16 S, SW17 X, SW18 LAlt, SW19 F2, SW2 Tilde, SW20 3, SW21 E, SW22 D, SW23 C, SW25 F3, SW26 4, SW27 R, SW28 F, SW29 V, SW3 Tab, SW31 F4, SW32 5, SW33 T, SW34 G, SW35 B, SW37 F5, SW38 6, SW39 Y, SW4 CapsLk, SW40 H, SW41 N, SW42 Space, SW43 F6, SW44 7, SW45 U, SW46 J, SW47 M, SW49 F7, SW5 LShift, SW50 8, SW51 I, SW52 K, SW53 ,, SW55 F8, SW56 9, SW57 O, SW58 L, SW59 ., SW6 LCtrl, SW61 F9, SW62 0, SW63 P, SW64 ;, SW65 /, SW66 AltGr, SW67 F10, SW68 -, SW69 [, SW70 ", SW71 RShift, SW72 RMeta, SW73 F11, SW74 =, SW75 ], SW76 ↲, SW78 Fn, SW79 F12, SW8 1, SW80 BkSpc, SW81 \, SW84 RCtrl, SW85 PrtSc, SW86 Ins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

Commit message: PCB: Move D5 and D80 over just a bit so they don't interfere with stabilizers
Parts:
- moved D5 1.17 mm to (42.3, 175.5)
- moved D80 0.76 mm to (287.5, 118.7)
Routing:
- net ColA: track 412.4 -> 413.7 mm
- net Net-(D5-Pad2): track 11.9 -> 13.1 mm
- net ColN: track 157.9 -> 158.8 mm
- net Net-(D80-Pad2): track 12.7 -> 13.4 mm
Changed lines of the file:
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@@
   )
   (footprint "RabidKeyboard:D_DO-35_SOD27_P7.62mm_Horizontal" (layer "F.Cu")
-    (at 43.434 175.514 90)
+    (at 42.2656 175.514 90)
     (descr "Diode, DO-35_SOD27 series, Axial, Horizontal, pin pitch=7.62mm, , length*diameter=4*2mm^2, , http://www.diodes.com/_files/packages/DO-35.pdf")
     (tags "Diode DO-35_SOD27 series Axial Horizontal pin pitch 7.62mm  length 4mm diameter 2mm")
@@
   )
   (footprint "RabidKeyboard:D_DO-35_SOD27_P7.62mm_Horizontal" (layer "F.Cu")
-    (at 288.29 118.745 90)
+    (at 287.528 118.7196 90)
     (descr "Diode, DO-35_SOD27 series, Axial, Horizontal, pin pitch=7.62mm, , length*diameter=4*2mm^2, , http://www.diodes.com/_files/packages/DO-35.pdf")
     (tags "Diode DO-35_SOD27 series Axial Horizontal pin pitch 7.62mm  length 4mm diameter 2mm")
@@
   (segment (start 106.521169 135.346449) (end 103.028828 135.34645) (width 0.3) (layer "F.Cu") (net 1))
   (segment (start 107.13568 135.96096) (end 106.521169 135.346449) (width 0.3) (layer "F.Cu") (net 1))
-  (segment (start 43.434 156.718) (end 44.683511 157.967511) (width 0.3) (layer "B.Cu") (net 1))
-  (segment (start 44.683511 157.967511) (end 44.683511 174.264489) (width 0.3) (layer "B.Cu") (net 1))
+  (segment (start 44.236645 173.542955) (end 42.2656 175.514) (width 0.3) (layer "B.Cu") (net 1))
   (segment (start 41.037479 111.149499) (end 41.037479 134.763479) (width 0.3) (layer "B.Cu") (net 1))
   (segment (start 48.808978 103.378) (end 41.037479 111.149499) (width 0.3) (layer "B.Cu") (net 1))
   (segment (start 41.037479 134.763479) (end 43.18 136.906) (width 0.3) (layer "B.Cu") (net 1))
   (segment (start 44.28 136.906) (end 44.683511 137.309511) (width 0.3) (layer "B.Cu") (net 1))
-  (segment (start 44.683511 174.264489) (end 43.434 175.514) (width 0.3) (layer "B.Cu") (net 1))
   (segment (start 44.683511 155.468489) (end 43.434 156.718) (width 0.3) (layer "B.Cu") (net 1))
   (segment (start 44.683511 137.309511) (end 44.683511 155.468489) (width 0.3) (layer "B.Cu") (net 1))
-  (segment (start 58.186489 184.698978) (end 58.186489 193.568489) (width 0.3) (layer "B.Cu") (net 1))
+  (segment (start 42.2656 175.514) (end 49.001511 175.514) (width 0.3) (layer "B.Cu") (net 1))
+  (segment (start 43.434 156.718) (end 44.236645 157.520645) (width 0.3) (layer "B.Cu") (net 1))
   (segment (start 43.18 136.906) (end 44.28 136.906) (width 0.3) (layer "B.Cu") (net 1))
+  (segment (start 44.236645 157.520645) (end 44.236645 173.542955) (width 0.3) (layer "B.Cu") (net 1))
   (segment (start 58.186489 193.568489) (end 59.436 194.818) (width 0.3) (layer "B.Cu") (net 1))
   (segment (start 57.404 97.282) (end 51.308 103.378) (width 0.3) (layer "B.Cu") (net 1))
   (segment (start 51.308 103.378) (end 48.808978 103.378) (width 0.3) (layer "B.Cu") (net 1))
+  (segment (start 58.186489 184.698978) (end 58.186489 193.568489) (width 0.3) (layer "B.Cu") (net 1))
   (segment (start 57.404 90.678) (end 57.404 97.282) (width 0.3) (layer "B.Cu") (net 1))
   (segment (start 49.001511 175.514) (end 58.186489 184.698978) (width 0.3) (layer "B.Cu") (net 1))
-  (segment (start 43.434 175.514) (end 49.001511 175.514) (width 0.3) (layer "B.Cu") (net 1))
   (segment (start 44.196 82.931) (end 57.404 82.931) (width 0.3) (layer "F.Cu") (net 2))
   (segment (start 43.688 103.378) (end 43.688 110.998) (width 0.3) (layer "F.Cu") (net 3))
   (segment (start 43.18 130.048) (end 48.4124 130.048) (width 0.3) (layer "F.Cu") (net 4))
   (segment (start 43.434 149.098) (end 50.8 149.098) (width 0.3) (layer "F.Cu") (net 5))
-  (segment (start 43.434 167.894) (end 55.3212 167.894) (width 0.3) (layer "F.Cu") (net 6))
+  (segment (start 42.2656 167.894) (end 55.372 167.894) (width 0.3) (layer "F.Cu") (net 6))
   (segment (start 46.3804 187.198) (end 59.436 187.198) (width 0.3) (layer "F.Cu") (net 7))
   (segment (start 311.17056 148.22956) (end 311.17056 147.04541) (width 0.3) (layer "F.Cu") (net 8))
@@
   (segment (start 281.686 183.420958) (end 281.575479 183.531479) (width 0.3) (layer "B.Cu") (net 82))
   (segment (start 304.8 83.058) (end 310.515 83.058) (width 0.3) (layer "F.Cu") (net 83))
-  (segment (start 288.29 111.125) (end 300.9646 111.125) (width 0.3) (layer "F.Cu") (net 84))
+  (segment (start 287.528 111.0996) (end 300.9392 111.0996) (width 0.3) (layer "F.Cu") (net 84))
   (segment (start 305.7652 130.2004) (end 298.4754 130.2004) (width 0.3) (layer "F.Cu") (net 85))
   (segment (start 300.355 187.325) (end 308.2036 187.325) (width 0.3) (layer "F.Cu") (net 86))
@@
   (via (at 299.212 183.642) (size 0.8) (drill 0.4) (layers "F.Cu" "B.Cu") (net 87))
   (segment (start 295.656 163.379741) (end 295.656 140.589) (width 0.3) (layer "B.Cu") (net 87))
-  (segment (start 288.29 118.745) (end 288.29 121.782076) (width 0.3) (layer "B.Cu") (net 87))
   (segment (start 299.105489 177.652511) (end 300.424259 176.333741) (width 0.3) (layer "B.Cu") (net 87))
   (segment (start 300.424259 168.148) (end 295.656 163.379741) (width 0.3) (layer "B.Cu") (net 87))
-  (segment (start 295.402 128.894076) (end 295.402 135.382) (width 0.3) (layer "B.Cu") (net 87))
-  (segment (start 288.29 121.782076) (end 295.402 128.894076) (width 0.3) (layer "B.Cu") (net 87))
   (segment (start 299.105489 193.695489) (end 299.105489 183.240511) (width 0.3) (layer "B.Cu") (net 87))
   (segment (start 299.105489 183.240511) (end 299.105489 177.652511) (width 0.3) (layer "B.Cu") (net 87))
   (segment (start 297.18 92.71) (end 290.068 99.822) (width 0.3) (layer "B.Cu") (net 87))
   (segment (start 295.656 140.589) (end 298.45 137.795) (width 0.3) (layer "B.Cu") (net 87))
+  (segment (start 287.528 118.7196) (end 287.528 121.92) (width 0.3) (layer "B.Cu") (net 87))
+  (segment (start 297.2308 136.5758) (end 298.45 137.795) (width 0.3) (layer "B.Cu") (net 87))
   (segment (start 300.424259 176.333741) (end 300.424259 168.148) (width 0.3) (layer "B.Cu") (net 87))
+  (segment (start 287.528 118.7196) (end 290.068 116.1796) (width 0.3) (layer "B.Cu") (net 87))
+  (segment (start 297.2308 131.6228) (end 297.2308 136.5758) (width 0.3) (layer "B.Cu") (net 87))
+  (segment (start 287.528 121.92) (end 297.2308 131.6228) (width 0.3) (layer "B.Cu") (net 87))
+  (segment (start 290.068 116.1796) (end 290.068 99.822) (width 0.3) (layer "B.Cu") (net 87))
   (segment (start 300.355 194.945) (end 299.105489 193.695489) (width 0.3) (layer "B.Cu") (net 87))
   (segment (start 299.212 183.347022) (end 299.105489 183.240511) (width 0.3) (layer "B.Cu") (net 87))
-  (segment (start 290.068 99.822) (end 290.068 116.967) (width 0.3) (layer "B.Cu") (net 87))
   (segment (start 302.768 92.71) (end 297.18 92.71) (width 0.3) (layer "B.Cu") (net 87))
-  (segment (start 295.402 135.382) (end 297.815 137.795) (width 0.3) (layer "B.Cu") (net 87))
   (segment (start 299.212 183.642) (end 299.212 183.347022) (width 0.3) (layer "B.Cu") (net 87))
-  (segment (start 290.068 116.967) (end 288.29 118.745) (width 0.3) (layer "B.Cu") (net 87))
   (segment (start 304.8 90.678) (end 302.768 92.71) (width 0.3) (layer "B.Cu") (net 87))
   (segment (start 328.93 83.058) (end 334.645 83.058) (width 0.3) (layer "F.Cu") (net 88))

Commit message: PCB: Swap Reset and BootSel button silkscreens.
Parts:
- SW103: value BootSel -> Reset
- SW104: value Reset -> BootSel
Changed lines of the file:
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@@
       (effects (font (size 1 1) (thickness 0.15)) (justify mirror))
     )
-    (fp_text value "BootSel" (at 3.504 -6.822) (layer "B.Fab")
+    (fp_text value "Reset" (at 3.504 -6.822) (layer "B.Fab")
       (effects (font (size 1 1) (thickness 0.15)) (justify mirror))
     )
@@
       (effects (font (size 1 1) (thickness 0.15)) (justify mirror))
     )
-    (fp_text value "Reset" (at 3.556 -6.822) (layer "B.Fab")
+    (fp_text value "BootSel" (at 3.556 -6.822) (layer "B.Fab")
       (effects (font (size 1 1) (thickness 0.15)) (justify mirror))
     )
@@
     (effects (font (size 1.5 1.5) (thickness 0.3)) (justify right mirror))
   )
-  (gr_text "Reset" (at 260.604 103.632) (layer "B.SilkS")
+  (gr_text "Reset" (at 247.65 103.632) (layer "B.SilkS")
     (effects (font (size 1 1) (thickness 0.15)) (justify mirror))
   )
@@
     (effects (font (size 1.5 1.5) (thickness 0.3)) (justify right mirror))
   )
-  (gr_text "BootSel" (at 247.65 103.632) (layer "B.SilkS")
+  (gr_text "BootSel" (at 260.604 103.632) (layer "B.SilkS")
     (effects (font (size 1 1) (thickness 0.15)) (justify mirror))
   )
