File: usb_costar/RabidUsb_costar.kicad_pcb (KiCad board)
At the start: 2 copper layers, 50 x 18 mm, 18 parts, among them J1 USB_C_Receptacle_USB2.0, J2 Conn_01x04, U1 SRV05-4

Commit message: USB: Update tooling holes to match what JLCPCB needed for assembly.
Parts:
- moved H7 8.55 mm to (141.4, 66.2)
- moved H8 1.22 mm to (114.8, 52.2)
Changed lines of the file:
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@@
   )
   (footprint "costar_footprints:ToolingHole_1.152mm" (layer "F.Cu")
-    (at 116 52.425)
+    (at 114.8 52.2)
     (descr "Mounting Hole 2.1mm, no annular")
     (tags "mounting hole 2.1mm no annular")
@@
   )
   (footprint "costar_footprints:ToolingHole_1.152mm" (layer "F.Cu")
-    (at 149.975 65.55)
+    (at 141.45 66.25)
     (descr "Mounting Hole 2.1mm, no annular")
     (tags "mounting hole 2.1mm no annular")

Commit message: USB: More ground plane between VCC and D+/D-.
Changed lines of the file:
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@@
   (segment (start 136.05 65.15) (end 137.4875 65.15) (width 0.875) (layer "F.Cu") (net 9))
   (segment (start 129.7 63.298896) (end 129.7 65.061396) (width 0.6) (layer "F.Cu") (net 10))
-  (segment (start 128.561396 65.111396) (end 125.425 61.975) (width 0.875) (layer "F.Cu") (net 10))
-  (segment (start 125.425 61.975) (end 113.475 61.975) (width 0.875) (layer "F.Cu") (net 10))
+  (segment (start 129.75 65.111396) (end 124.061396 65.111396) (width 0.875) (layer "F.Cu") (net 10))
+  (segment (start 120.925 61.975) (end 113.475 61.975) (width 0.875) (layer "F.Cu") (net 10))
   (segment (start 129.7 65.061396) (end 129.75 65.111396) (width 0.875) (layer "F.Cu") (net 10))
-  (segment (start 129.75 65.111396) (end 128.561396 65.111396) (width 0.875) (layer "F.Cu") (net 10))
+  (segment (start 124.061396 65.111396) (end 120.925 61.975) (width 0.875) (layer "F.Cu") (net 10))
   (segment (start 129.788604 65.15) (end 129.75 65.111396) (width 0.875) (layer "F.Cu") (net 10))
   (segment (start 132.75 65.15) (end 129.788604 65.15) (width 0.875) (layer "F.Cu") (net 10))
