File: usb_costar/RabidUsb_costar.kicad_pcb (KiCad board)
At the start: 2 copper layers, 50 x 18 mm, 18 parts, among them J1 USB_C_Receptacle_USB2.0, J2 Conn_01x04, U1 SRV05-4

Commit message: USB: Add ferrite beads to usb_costar board as well.
Parts:
- added FB1: FerriteBead_Small, Inductor_SMD:L_0805_2012Metric, F.Cu at (117.0, 62.0)
- added FB2: FerriteBead_Small, Inductor_SMD:L_0805_2012Metric, F.Cu at (117.0, 56.0)
- moved FID1 3.93 mm to (122.3, 52.5)
Connections:
- J2 pad 1: VCC -> Net-(J2-Pad1)
- J2 pad 4: GND -> Net-(J2-Pad4)
Routing:
- net VCC: track 22.4 -> 17.8 mm
- net Net-(J2-Pad4): track 0.00 -> 2.51 mm
- net Net-(J2-Pad1): track 0.00 -> 2.51 mm
- net GND: vias 40 -> 43
Changed lines of the file:
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@@
   (net 11 "unconnected-(U1-Pad3)")
   (net 12 "unconnected-(U1-Pad4)")
+  (net 13 "Net-(J2-Pad1)")
+  (net 14 "Net-(J2-Pad4)")
   (footprint "costar_footprints:MountingHole_2.5mm_Pad_1mm" (layer "F.Cu")
     (at 155.575 52.425)
@@
   )
   (footprint "Fiducial:Fiducial_1mm_Mask2mm" (layer "F.Cu")
-    (at 118.625 53.95)
+    (at 122.3 52.55)
     (descr "Circular Fiducial, 1mm bare copper, 2mm soldermask opening (Level A)")
     (tags "fiducial")
@@
     )
   )
+  (footprint "Inductor_SMD:L_0805_2012Metric" (layer "F.Cu")
+    (at 117.05 55.975)
+    (descr "Inductor SMD 0805 (2012 Metric), square (rectangular) end terminal, IPC_7351 nominal, (Body size source: IPC-SM-782 page 80, https://www.pcb-3d.com/wordpress/wp-content/uploads/ipc-sm-782a_amendment_1_and_2.pdf), generated with kicad-footprint-generator")
+    (tags "inductor")
+    (property "LCSC" " C67451")
+    (property "Sheetfile" "RabidUsb_costar.kicad_sch")
+    (property "Sheetname" "")
+    (attr smd)
+    (fp_text reference "FB2" (at -0.5125 -1.425) (layer "F.SilkS")
+      (effects (font (size 1 1) (thickness 0.15)))
+    )
+    (fp_text value "FerriteBead_Small" (at 0 1.55) (layer "F.Fab") hide
+      (effects (font (size 1 1) (thickness 0.15)))
+    )
+    (fp_text user "${REFERENCE}" (at 0 0) (layer "F.Fab")
+      (effects (font (size 0.5 0.5) (thickness 0.08)))
+    )
+    (fp_line (start -0.399622 -0.56) (end 0.399622 -0.56) (layer "F.SilkS") (width 0.12))
+    (fp_line (start -0.399622 0.56) (end 0.399622 0.56) (layer "F.SilkS") (width 0.12))
+    (fp_line (start -1.75 -0.85) (end 1.75 -0.85) (layer "F.CrtYd") (width 0.05))
+    (fp_line (start 1.75 0.85) (end -1.75 0.85) (layer "F.CrtYd") (width 0.05))
+    (fp_line (start 1.75 -0.85) (end 1.75 0.85) (layer "F.CrtYd") (width 0.05))
+    (fp_line (start -1.75 0.85) (end -1.75 -0.85) (layer "F.CrtYd") (width 0.05))
+    (fp_line (start 1 -0.45) (end 1 0.45) (layer "F.Fab") (width 0.1))
+    (fp_line (start 1 0.45) (end -1 0.45) (layer "F.Fab") (width 0.1))
+    (fp_line (start -1 -0.45) (end 1 -0.45) (layer "F.Fab") (width 0.1))
+    (fp_line (start -1 0.45) (end -1 -0.45) (layer "F.Fab") (width 0.1))
+    (pad "1" smd roundrect (at -1.0625 0) (size 0.875 1.2) (layers "F.Cu" "F.Paste" "F.Mask") (roundrect_rratio 0.25)
+      (net 14 "Net-(J2-Pad4)") (pintype "passive"))
+    (pad "2" smd roundrect (at 1.0625 0) (size 0.875 1.2) (layers "F.Cu" "F.Paste" "F.Mask") (roundrect_rratio 0.25)
+      (net 2 "GND") (pintype "passive"))
+    (model "${KICAD6_3DMODEL_DIR}/Inductor_SMD.3dshapes/L_0805_2012Metric.wrl"
+      (offset (xyz 0 0 0))
+      (scale (xyz 1 1 1))
+      (rotate (xyz 0 0 0))
+    )
+  )
   (footprint "costar_footprints:MountingHole_2.5mm_Pad_1mm" (layer "F.Cu")
     (at 110.425 52.425)
@@
     )
   )
+  (footprint "Inductor_SMD:L_0805_2012Metric" (layer "F.Cu")
+    (at 117.05 61.975 180)
+    (descr "Inductor SMD 0805 (2012 Metric), square (rectangular) end terminal, IPC_7351 nominal, (Body size source: IPC-SM-782 page 80, https://www.pcb-3d.com/wordpress/wp-content/uploads/ipc-sm-782a_amendment_1_and_2.pdf), generated with kicad-footprint-generator")
+    (tags "inductor")
+    (property "LCSC" " C67451")
+    (property "Sheetfile" "RabidUsb_costar.kicad_sch")
+    (property "Sheetname" "")
+    (attr smd)
+    (fp_text reference "FB1" (at -0.9 -1.525) (layer "F.SilkS")
+      (effects (font (size 1 1) (thickness 0.15)))
+    )
+    (fp_text value "FerriteBead_Small" (at 0 1.55) (layer "F.Fab") hide
+      (effects (font (size 1 1) (thickness 0.15)))
+    )
+    (fp_text user "${REFERENCE}" (at 0 0) (layer "F.Fab")
+      (effects (font (size 0.5 0.5) (thickness 0.08)))
+    )
+    (fp_line (start -0.399622 -0.56) (end 0.399622 -0.56) (layer "F.SilkS") (width 0.12))
+    (fp_line (start -0.399622 0.56) (end 0.399622 0.56) (layer "F.SilkS") (width 0.12))
+    (fp_line (start -1.75 -0.85) (end 1.75 -0.85) (layer "F.CrtYd") (width 0.05))
+    (fp_line (start 1.75 -0.85) (end 1.75 0.85) (layer "F.CrtYd") (width 0.05))
+    (fp_line (start -1.75 0.85) (end -1.75 -0.85) (layer "F.CrtYd") (width 0.05))
+    (fp_line (start 1.75 0.85) (end -1.75 0.85) (layer "F.CrtYd") (width 0.05))
+    (fp_line (start 1 -0.45) (end 1 0.45) (layer "F.Fab") (width 0.1))
+    (fp_line (start -1 -0.45) (end 1 -0.45) (layer "F.Fab") (width 0.1))
+    (fp_line (start 1 0.45) (end -1 0.45) (layer "F.Fab") (width 0.1))
+    (fp_line (start -1 0.45) (end -1 -0.45) (layer "F.Fab") (width 0.1))
+    (pad "1" smd roundrect (at -1.0625 0 180) (size 0.875 1.2) (layers "F.Cu" "F.Paste" "F.Mask") (roundrect_rratio 0.25)
+      (net 10 "VCC") (pintype "passive"))
+    (pad "2" smd roundrect (at 1.0625 0 180) (size 0.875 1.2) (layers "F.Cu" "F.Paste" "F.Mask") (roundrect_rratio 0.25)
+      (net 13 "Net-(J2-Pad1)") (pintype "passive"))
+    (model "${KICAD6_3DMODEL_DIR}/Inductor_SMD.3dshapes/L_0805_2012Metric.wrl"
+      (offset (xyz 0 0 0))
+      (scale (xyz 1 1 1))
+      (rotate (xyz 0 0 0))
+    )
+  )
   (footprint "costar_footprints:ToolingHole_1.152mm" (layer "F.Cu")
     (at 141.45 66.25)
@@
       (net 2 "GND") (pinfunction "VN") (pintype "passive"))
     (pad "3" smd roundrect (at -1.1375 0.95 270) (size 1.325 0.6) (layers "F.Cu" "F.Paste" "F.Mask") (roundrect_rratio 0.25)
-      (net 11 "unconnected-(U1-Pad3)") (pinfunction "IO2") (pintype "passive"))
+      (net 11 "unconnected-(U1-Pad3)") (pinfunction "IO2") (pintype "passive+no_connect"))
     (pad "4" smd roundrect (at 1.1375 0.95 270) (size 1.325 0.6) (layers "F.Cu" "F.Paste" "F.Mask") (roundrect_rratio 0.25)
-      (net 12 "unconnected-(U1-Pad4)") (pinfunction "IO3") (pintype "passive"))
+      (net 12 "unconnected-(U1-Pad4)") (pinfunction "IO3") (pintype "passive+no_connect"))
     (pad "5" smd roundrect (at 1.1375 0 270) (size 1.325 0.6) (layers "F.Cu" "F.Paste" "F.Mask") (roundrect_rratio 0.25)
       (net 10 "VCC") (pinfunction "VP") (pintype "passive"))
@@
     (property "Sheetname" "")
     (property "exclude_from_bom" "")
-    (attr through_hole)
+    (attr through_hole exclude_from_bom)
     (fp_text reference "J2" (at 0 2.06 180) (layer "B.SilkS")
       (effects (font (size 1 1) (thickness 0.15)) (justify mirror))
@@
     (fp_line (start 1 -7) (end -1 -7) (layer "B.Fab") (width 0.1))
     (pad "1" thru_hole rect (at 0 0) (size 1.35 1.35) (drill 0.8) (layers *.Cu *.Mask)
-      (net 10 "VCC") (pinfunction "Pin_1") (pintype "passive"))
+      (net 13 "Net-(J2-Pad1)") (pinfunction "Pin_1") (pintype "passive"))
     (pad "2" thru_hole oval (at 0 -2) (size 1.35 1.35) (drill 0.8) (layers *.Cu *.Mask)
       (net 5 "/USB_D-") (pinfunction "Pin_2") (pintype "passive"))
@@
       (net 4 "/USB_D+") (pinfunction "Pin_3") (pintype "passive"))
     (pad "4" thru_hole oval (at 0 -6) (size 1.35 1.35) (drill 0.8) (layers *.Cu *.Mask)
-      (net 2 "GND") (pinfunction "Pin_4") (pintype "passive"))
+      (net 14 "Net-(J2-Pad4)") (pinfunction "Pin_4") (pintype "passive"))
     (model "${KICAD6_3DMODEL_DIR}/Connector_PinHeader_2.00mm.3dshapes/PinHeader_1x04_P2.00mm_Horizontal.wrl"
       (offset (xyz 0 -6 0))
@@
   (via (at 116 60.5) (size 0.8) (drill 0.4) (layers "F.Cu" "B.Cu") (free) (net 2))
   (via (at 150 63.5) (size 0.8) (drill 0.4) (layers "F.Cu" "B.Cu") (free) (net 2))
+  (via (at 139.75 61.825) (size 0.8) (drill 0.4) (layers "F.Cu" "B.Cu") (free) (net 2))
   (via (at 120 60.5) (size 0.8) (drill 0.4) (layers "F.Cu" "B.Cu") (free) (net 2))
   (via (at 120 63.5) (size 0.8) (drill 0.4) (layers "F.Cu" "B.Cu") (free) (net 2))
@@
   (via (at 140 54) (size 0.8) (drill 0.4) (layers "F.Cu" "B.Cu") (free) (net 2))
   (via (at 130.55 51.15) (size 0.8) (drill 0.4) (layers "F.Cu" "B.Cu") (free) (net 2))
+  (via (at 137.65 61.825) (size 0.8) (drill 0.4) (layers "F.Cu" "B.Cu") (free) (net 2))
   (via (at 150 57.5) (size 0.8) (drill 0.4) (layers "F.Cu" "B.Cu") (free) (net 2))
   (via (at 145 51.15) (size 0.8) (drill 0.4) (layers "F.Cu" "B.Cu") (free) (net 2))
+  (via (at 120.2 54) (size 0.8) (drill 0.4) (layers "F.Cu" "B.Cu") (free) (net 2))
   (via (at 140 57.5) (size 0.8) (drill 0.4) (layers "F.Cu" "B.Cu") (free) (net 2))
   (via (at 120 66.5) (size 0.8) (drill 0.4) (layers "F.Cu" "B.Cu") (free) (net 2))
@@
   (segment (start 129.7 63.298896) (end 129.7 65.061396) (width 0.6) (layer "F.Cu") (net 10))
   (segment (start 129.75 65.111396) (end 124.061396 65.111396) (width 0.875) (layer "F.Cu") (net 10))
-  (segment (start 120.925 61.975) (end 113.475 61.975) (width 0.875) (layer "F.Cu") (net 10))
+  (segment (start 120.925 61.975) (end 118.1125 61.975) (width 0.875) (layer "F.Cu") (net 10))
   (segment (start 129.7 65.061396) (end 129.75 65.111396) (width 0.875) (layer "F.Cu") (net 10))
   (segment (start 124.061396 65.111396) (end 120.925 61.975) (width 0.875) (layer "F.Cu") (net 10))
   (segment (start 129.788604 65.15) (end 129.75 65.111396) (width 0.875) (layer "F.Cu") (net 10))
   (segment (start 132.75 65.15) (end 129.788604 65.15) (width 0.875) (layer "F.Cu") (net 10))
+  (segment (start 115.9875 61.975) (end 113.475 61.975) (width 0.875) (layer "F.Cu") (net 13))
+  (segment (start 115.9875 55.975) (end 113.475 55.975) (width 0.875) (layer "F.Cu") (net 14))
   (zone (net 1) (net_name "VBUS") (layer "F.Cu") (name "VBUS_CONN") (hatch edge 0.508)
     (priority 1)
