File: usb_costar/RabidUsb_costar.kicad_sch (KiCad schematic)
At the start: 18 parts, among them J1 USB_C_Receptacle_USB2.0, J2 Conn_01x04, U1 SRV05-4

Commit message: USB: Add ferrite beads to usb_costar board as well.
Parts:
- added FB1, FB2: FerriteBead_Small, Inductor_SMD:L_0805_2012Metric, symbol Device:FerriteBead_Small
Connections:
- net GND: now also FB2.2; no longer J2.4 (Pin_4)
- net VCC: now also FB1.1; no longer J2.1 (Pin_1)
- new net: FB2.1, J2.4 (Pin_4)
- new net: FB1.2, J2.1 (Pin_1)
Changed lines of the file:
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@@
   (junction (at 71.12 36.83) (diameter 0) (color 0 0 0 0)
-  )
-  (junction (at 172.72 54.61) (diameter 0) (color 0 0 0 0)
   )
   (no_connect (at 55.88 59.69))
@@
     (stroke (width 0) (type default) (color 0 0 0 0))
   )
-  (wire (pts (xy 177.8 40.64) (xy 172.72 40.64))
-    (stroke (width 0) (type default) (color 0 0 0 0))
-  )
   (wire (pts (xy 40.64 68.58) (xy 40.64 67.31))
     (stroke (width 0) (type solid) (color 0 0 0 0))
@@
     (stroke (width 0) (type solid) (color 0 0 0 0))
   )
+  (wire (pts (xy 172.72 57.15) (xy 172.72 58.42))
+    (stroke (width 0) (type default) (color 0 0 0 0))
+  )
   (wire (pts (xy 55.88 46.99) (xy 57.15 46.99))
     (stroke (width 0) (type solid) (color 0 0 0 0))
@@
     (stroke (width 0) (type solid) (color 0 0 0 0))
   )
-  (wire (pts (xy 172.72 54.61) (xy 172.72 55.88))
-    (stroke (width 0) (type default) (color 0 0 0 0))
-  )
   (wire (pts (xy 104.14 45.72) (xy 114.3 45.72))
     (stroke (width 0) (type default) (color 0 0 0 0))
@@
     (stroke (width 0) (type solid) (color 0 0 0 0))
   )
-  (wire (pts (xy 172.72 35.56) (xy 172.72 40.64))
-    (stroke (width 0) (type default) (color 0 0 0 0))
-  )
   (wire (pts (xy 87.63 25.4) (xy 87.63 29.21))
     (stroke (width 0) (type default) (color 0 0 0 0))
@@
     (stroke (width 0) (type default) (color 0 0 0 0))
   )
+  (wire (pts (xy 172.72 38.1) (xy 172.72 40.64))
+    (stroke (width 0) (type default) (color 0 0 0 0))
+  )
+  (wire (pts (xy 172.72 48.26) (xy 172.72 52.07))
+    (stroke (width 0) (type default) (color 0 0 0 0))
+  )
   (wire (pts (xy 55.88 25.4) (xy 55.88 29.21))
     (stroke (width 0) (type default) (color 0 0 0 0))
   )
+  (wire (pts (xy 172.72 31.75) (xy 172.72 33.02))
+    (stroke (width 0) (type default) (color 0 0 0 0))
+  )
   (wire (pts (xy 58.42 101.6) (xy 58.42 120.65))
     (stroke (width 0) (type default) (color 0 0 0 0))
@@
     (stroke (width 0) (type solid) (color 0 0 0 0))
   )
+  (wire (pts (xy 172.72 40.64) (xy 177.8 40.64))
+    (stroke (width 0) (type default) (color 0 0 0 0))
+  )
   (wire (pts (xy 58.42 95.25) (xy 58.42 101.6))
     (stroke (width 0) (type default) (color 0 0 0 0))
@@
   )
   (wire (pts (xy 139.7 45.72) (xy 144.78 45.72))
-    (stroke (width 0) (type default) (color 0 0 0 0))
-  )
-  (wire (pts (xy 172.72 48.26) (xy 172.72 54.61))
     (stroke (width 0) (type default) (color 0 0 0 0))
   )
@@
     )
   )
+  (symbol (lib_id "Device:FerriteBead_Small") (at 172.72 54.61 0) (unit 1)
+    (in_bom yes) (on_board yes) (fields_autoplaced)
+    (property "Reference" "FB2" (id 0) (at 175.26 54.5718 0)
+      (effects (font (size 1.27 1.27)) (justify left))
+    )
+    (property "Value" "FerriteBead_Small" (id 1) (at 175.26 55.8418 0)
+      (effects (font (size 1.27 1.27)) (justify left) hide)
+    )
+    (property "Footprint" "Inductor_SMD:L_0805_2012Metric" (id 2) (at 170.942 54.61 90)
+      (effects (font (size 1.27 1.27)) hide)
+    )
+    (property "Datasheet" "https://datasheet.lcsc.com/lcsc/1811061723_FH-Guangdong-Fenghua-Advanced-Tech-CBW201209U301T_C67451.pdf" (id 3) (at 172.72 54.61 0)
+      (effects (font (size 1.27 1.27)) hide)
+    )
+    (property "LCSC" " C67451" (id 4) (at 172.72 54.61 0)
+      (effects (font (size 1.27 1.27)) hide)
+    )
+    (pin "1")
+    (pin "2")
+  )
   (symbol (lib_id "Mechanical:MountingHole_Pad") (at 35.56 107.95 270) (unit 1)
     (in_bom no) (on_board yes) (fields_autoplaced)
@@
     )
   )
-  (symbol (lib_id "power:VCC") (at 172.72 35.56 0) (unit 1)
-    (in_bom yes) (on_board yes)
-    (property "Reference" "#PWR0107" (id 0) (at 172.72 39.37 0)
-      (effects (font (size 1.27 1.27)) hide)
-    )
-    (property "Value" "VCC" (id 1) (at 172.72 31.75 0))
-    (property "Footprint" "" (id 2) (at 172.72 35.56 0)
-      (effects (font (size 1.27 1.27)) hide)
-    )
-    (property "Datasheet" "" (id 3) (at 172.72 35.56 0)
+  (symbol (lib_id "power:VCC") (at 172.72 31.75 0) (unit 1)
+    (in_bom yes) (on_board yes)
+    (property "Reference" "#PWR0107" (id 0) (at 172.72 35.56 0)
+      (effects (font (size 1.27 1.27)) hide)
+    )
+    (property "Value" "VCC" (id 1) (at 172.72 27.94 0))
+    (property "Footprint" "" (id 2) (at 172.72 31.75 0)
+      (effects (font (size 1.27 1.27)) hide)
+    )
+    (property "Datasheet" "" (id 3) (at 172.72 31.75 0)
       (effects (font (size 1.27 1.27)) hide)
     )
@@
     (pin "6")
   )
+  (symbol (lib_id "Device:FerriteBead_Small") (at 172.72 35.56 0) (unit 1)
+    (in_bom yes) (on_board yes) (fields_autoplaced)
+    (property "Reference" "FB1" (id 0) (at 175.26 35.5218 0)
+      (effects (font (size 1.27 1.27)) (justify left))
+    )
+    (property "Value" "FerriteBead_Small" (id 1) (at 175.26 36.7918 0)
+      (effects (font (size 1.27 1.27)) (justify left) hide)
+    )
+    (property "Footprint" "Inductor_SMD:L_0805_2012Metric" (id 2) (at 170.942 35.56 90)
+      (effects (font (size 1.27 1.27)) hide)
+    )
+    (property "Datasheet" "https://datasheet.lcsc.com/lcsc/1811061723_FH-Guangdong-Fenghua-Advanced-Tech-CBW201209U301T_C67451.pdf" (id 3) (at 172.72 35.56 0)
+      (effects (font (size 1.27 1.27)) hide)
+    )
+    (property "LCSC" " C67451" (id 4) (at 172.72 35.56 0)
+      (effects (font (size 1.27 1.27)) hide)
+    )
+    (pin "1")
+    (pin "2")
+  )
   (symbol (lib_id "Mechanical:MountingHole_Pad") (at 35.56 95.25 270) (unit 1)
     (in_bom no) (on_board yes) (fields_autoplaced)
@@
     (pin "1")
   )
-  (symbol (lib_id "power:GND") (at 172.72 54.61 0) (unit 1)
-    (in_bom yes) (on_board yes)
-    (property "Reference" "#PWR08" (id 0) (at 172.72 60.96 0)
-      (effects (font (size 1.27 1.27)) hide)
-    )
-    (property "Value" "GND" (id 1) (at 172.72 58.42 0))
-    (property "Footprint" "" (id 2) (at 172.72 54.61 0))
-    (property "Datasheet" "" (id 3) (at 172.72 54.61 0))
+  (symbol (lib_id "power:GND") (at 172.72 58.42 0) (unit 1)
+    (in_bom yes) (on_board yes)
+    (property "Reference" "#PWR08" (id 0) (at 172.72 64.77 0)
+      (effects (font (size 1.27 1.27)) hide)
+    )
+    (property "Value" "GND" (id 1) (at 172.72 62.23 0))
+    (property "Footprint" "" (id 2) (at 172.72 58.42 0))
+    (property "Datasheet" "" (id 3) (at 172.72 58.42 0))
     (pin "1")
   )
@@
       (reference "F1") (unit 1) (value "500mA") (footprint "Fuse:Fuse_1812_4532Metric")
     )
+    (path "/d0385045-2f04-4b10-8a4f-831056275697"
+      (reference "FB1") (unit 1) (value "FerriteBead_Small") (footprint "Inductor_SMD:L_0805_2012Metric")
+    )
+    (path "/3f7d00b9-25d3-4bcc-a8f5-a4b9bd919b65"
+      (reference "FB2") (unit 1) (value "FerriteBead_Small") (footprint "Inductor_SMD:L_0805_2012Metric")
+    )
     (path "/732031ed-0f98-4524-ab12-56a5343cf649"
